Commit message: change for upper body controller

File: src/engineai_ros2/urdf/pm_v2_ros2_control.xacro (robot description, xacro)
@@ -8,131 +8,97 @@
         <param name="example_param_hw_stop_duration_sec">3.0</param>
         <param name="example_param_hw_slowdown">100</param>
-	<!-- Defaults -->
-	<param name="default_stiffness">20.0</param>
-	<param name="default_damping">1.0</param>
-	<!-- Per-joint overrides: "JOINT_NAME=value,JOINT_NAME=value,..." -->
-	<param name="stiffness_by_joint">
-	  J12_WAIST_YAW=200,J13_SHOULDER_PITCH_L=250,J14_SHOULDER_ROLL_L=250,J15_SHOULDER_YAW_L=250,J16_ELBOW_PITCH_L=250,J17_ELBOW_YAW_L=250,J18_SHOULDER_PITCH_R=250,J19_SHOULDER_ROLL_R=250,J20_SHOULDER_YAW_R=250,J21_ELBOW_PITCH_R=250,J22_ELBOW_YAW_R=250,J23_HEAD_YAW=100
-	</param>
+	<!-- stiffness=80: high enough to move joints via incremental JTC commands,
+	     low enough to avoid aggressive snapping from rqt goal preemption.
+	     (examples use 20.0 because they send large single-step targets;
+	      JTC sends fine increments so a higher value is needed.) -->
+	<param name="default_stiffness">80.0</param>
+	<param name="default_damping">2.0</param>
       </hardware>
+      <!-- Left leg joints (state-only — controlled by onboard RL locomotion controller) -->
       <joint name="J00_HIP_PITCH_L">
-	<command_interface name="position"/>
 	<state_interface name="position"/>
-	<!-- <state_interface name="velocity"/> -->
       </joint>
       <joint name="J01_HIP_ROLL_L">
-	<command_interface name="position"/>
 	<state_interface name="position"/>
-	<!-- <state_interface name="velocity"/> -->
       </joint>
       <joint name="J02_HIP_YAW_L">
-	<command_interface name="position"/>
 	<state_interface name="position"/>
-	<!-- <state_interface name="velocity"/> -->
       </joint>
       <joint name="J03_KNEE_PITCH_L">
-	<command_interface name="position"/>
 	<state_interface name="position"/>
-	<!-- <state_interface name="velocity"/> -->
       </joint>
       <joint name="J04_ANKLE_PITCH_L">
-	<command_interface name="position"/>
 	<state_interface name="position"/>
-	<!-- <state_interface name="velocity"/> -->
       </joint>
       <joint name="J05_ANKLE_ROLL_L">
-	<command_interface name="position"/>
 	<state_interface name="position"/>
-	<!-- <state_interface name="velocity"/> -->
       </joint>
+      <!-- Right leg joints (state-only — controlled by onboard RL locomotion controller) -->
       <joint name="J06_HIP_PITCH_R">
-	<command_interface name="position"/>
 	<state_interface name="position"/>
-	<!-- <state_interface name="velocity"/> -->
       </joint>
       <joint name="J07_HIP_ROLL_R">
-	<command_interface name="position"/>
 	<state_interface name="position"/>
-	<!-- <state_interface name="velocity"/> -->
       </joint>
       <joint name="J08_HIP_YAW_R">
-	<command_interface name="position"/>
 	<state_interface name="position"/>
-	<!-- <state_interface name="velocity"/> -->
       </joint>
-      <joint  name="J09_KNEE_PITCH_R">
-	<command_interface name="position"/>
+      <joint name="J09_KNEE_PITCH_R">
 	<state_interface name="position"/>
-	<!-- <state_interface name="velocity"/> -->
       </joint>
       <joint name="J10_ANKLE_PITCH_R">
-	<command_interface name="position"/>
 	<state_interface name="position"/>
-	<!-- <state_interface name="velocity"/> -->
       </joint>
       <joint name="J11_ANKLE_ROLL_R">
-	<command_interface name="position"/>
 	<state_interface name="position"/>
-	<!-- <state_interface name="velocity"/> -->
       </joint>
+      <!-- Upper body joints (command + state) -->
       <joint name="J12_WAIST_YAW">
 	<command_interface name="position"/>
 	<state_interface name="position"/>
-	<!-- <state_interface name="velocity"/> -->
       </joint>
       <joint name="J13_SHOULDER_PITCH_L">
 	<command_interface name="position"/>
 	<state_interface name="position"/>
-	<!-- <state_interface name="velocity"/> -->
       </joint>
       <joint name="J14_SHOULDER_ROLL_L">
 	<command_interface name="position"/>
 	<state_interface name="position"/>
-	<!-- <state_interface name="velocity"/> -->
       </joint>
       <joint name="J15_SHOULDER_YAW_L">
 	<command_interface name="position"/>
 	<state_interface name="position"/>
-	<!-- <state_interface name="velocity"/> -->
       </joint>
       <joint name="J16_ELBOW_PITCH_L">
 	<command_interface name="position"/>
 	<state_interface name="position"/>
-	<!-- <state_interface name="velocity"/> -->
       </joint>
       <joint name="J17_ELBOW_YAW_L">
 	<command_interface name="position"/>
 	<state_interface name="position"/>
-	<!-- <state_interface name="velocity"/> -->
       </joint>
       <joint name="J18_SHOULDER_PITCH_R">
 	<command_interface name="position"/>
 	<state_interface name="position"/>
-	<!-- <state_interface name="velocity"/> -->
       </joint>
       <joint name="J19_SHOULDER_ROLL_R">
 	<command_interface name="position"/>
 	<state_interface name="position"/>
-	<!-- <state_interface name="velocity"/> -->
       </joint>
       <joint name="J20_SHOULDER_YAW_R">
 	<command_interface name="position"/>
 	<state_interface name="position"/>
-	<!-- <state_interface name="velocity"/> -->
       </joint>
       <joint name="J21_ELBOW_PITCH_R">
 	<command_interface name="position"/>
 	<state_interface name="position"/>
-	<!-- <state_interface name="velocity"/> -->
       </joint>
       <joint name="J22_ELBOW_YAW_R">
 	<command_interface name="position"/>
 	<state_interface name="position"/>
-	<!-- <state_interface name="velocity"/> -->
       </joint>
       <joint name="J23_HEAD_YAW">
 	<command_interface name="position"/>
 	<state_interface name="position"/>
-	<!-- <state_interface name="velocity"/> -->
       </joint>
     </ros2_control>
